File: FLC-148 - LED & Keypad panel/FLC-148 LED & Keypad panel.brd (EAGLE design)
At the start: 52 x 73.8 mm, 76 parts, among them IC1 MAX6818, IC2 MAX6818, IC3 NTGD3148NT1G, IC4 NTGD3148NT1G, IC5 STM32G071CBU6, IC6 ECS-480-10-33B-CKM-TR, J1 FTSH-107-01-L-DV-K-A

Commit message: start of rev.2 board - the LCD D/C signal wasn't routed - pulldown resistors are likely needed for LED gate control - boot0 likely needs to be tied to GND
Connections:
- net BACKLIGHT_GREEN_DRAIN renamed LCD_BACKLIGHT_GREEN_DRAIN
- net BACKLIGHT_IR_DRAIN renamed LCD_BACKLIGHT_IR_DRAIN
- net LED_BACKLIGHT_GREEN_GATE renamed LCD_BACKLIGHT_GREEN_GATE
- net LED_BACKLIGHT_IR_GATE renamed LCD_BACKLIGHT_IR_GATE
- net OLED_!D!/C renamed LCD_!D!/C
- net OLED_RST renamed LCD_RST
Changed lines of the file:
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@@
 <layers>
 <layer number="1" name="Top" color="4" fill="1" visible="yes" active="yes"/>
-<layer number="2" name="Route2" color="16" fill="1" visible="yes" active="yes"/>
+<layer number="2" name="Route2" color="16" fill="1" visible="no" active="yes"/>
 <layer number="3" name="Route3" color="17" fill="1" visible="no" active="no"/>
 <layer number="4" name="Route4" color="18" fill="1" visible="no" active="no"/>
@@
 <layer number="13" name="Route13" color="21" fill="1" visible="no" active="no"/>
 <layer number="14" name="Route14" color="22" fill="1" visible="no" active="no"/>
-<layer number="15" name="Route15" color="23" fill="1" visible="yes" active="yes"/>
-<layer number="16" name="Bottom" color="1" fill="1" visible="yes" active="yes"/>
+<layer number="15" name="Route15" color="23" fill="1" visible="no" active="yes"/>
+<layer number="16" name="Bottom" color="1" fill="1" visible="no" active="yes"/>
 <layer number="17" name="Pads" color="2" fill="1" visible="yes" active="yes"/>
 <layer number="18" name="Vias" color="2" fill="1" visible="yes" active="yes"/>
@@
 <layer number="20" name="Dimension" color="24" fill="1" visible="yes" active="yes"/>
 <layer number="21" name="tPlace" color="7" fill="1" visible="yes" active="yes"/>
-<layer number="22" name="bPlace" color="7" fill="1" visible="yes" active="yes"/>
+<layer number="22" name="bPlace" color="7" fill="1" visible="no" active="yes"/>
 <layer number="23" name="tOrigins" color="15" fill="1" visible="yes" active="yes"/>
-<layer number="24" name="bOrigins" color="15" fill="1" visible="yes" active="yes"/>
-<layer number="25" name="tNames" color="7" fill="1" visible="no" active="yes"/>
+<layer number="24" name="bOrigins" color="15" fill="1" visible="no" active="yes"/>
+<layer number="25" name="tNames" color="7" fill="1" visible="yes" active="yes"/>
 <layer number="26" name="bNames" color="7" fill="1" visible="no" active="yes"/>
 <layer number="27" name="tValues" color="7" fill="1" visible="no" active="yes"/>
 <layer number="28" name="bValues" color="7" fill="1" visible="no" active="yes"/>
-<layer number="29" name="tStop" color="7" fill="3" visible="no" active="yes"/>
+<layer number="29" name="tStop" color="7" fill="3" visible="yes" active="yes"/>
 <layer number="30" name="bStop" color="7" fill="6" visible="no" active="yes"/>
 <layer number="31" name="tCream" color="7" fill="4" visible="no" active="yes"/>
@@
 <layer number="38" name="bTest" color="7" fill="1" visible="no" active="yes"/>
 <layer number="39" name="tKeepout" color="4" fill="11" visible="yes" active="yes"/>
-<layer number="40" name="bKeepout" color="1" fill="11" visible="yes" active="yes"/>
+<layer number="40" name="bKeepout" color="1" fill="11" visible="no" active="yes"/>
 <layer number="41" name="tRestrict" color="4" fill="10" visible="yes" active="yes"/>
-<layer number="42" name="bRestrict" color="1" fill="10" visible="yes" active="yes"/>
+<layer number="42" name="bRestrict" color="1" fill="10" visible="no" active="yes"/>
 <layer number="43" name="vRestrict" color="2" fill="10" visible="yes" active="yes"/>
 <layer number="44" name="Drills" color="7" fill="1" visible="no" active="yes"/>
@@
 <layer number="50" name="dxf" color="7" fill="1" visible="no" active="no"/>
 <layer number="51" name="tDocu" color="7" fill="1" visible="yes" active="yes"/>
-<layer number="52" name="bDocu" color="7" fill="1" visible="yes" active="yes"/>
+<layer number="52" name="bDocu" color="7" fill="1" visible="no" active="yes"/>
 <layer number="53" name="tGND_GNDA" color="7" fill="1" visible="no" active="no"/>
 <layer number="54" name="bGND_GNDA" color="7" fill="1" visible="no" active="no"/>
@@
 <wire x1="41.29" y1="37.79" x2="41.29" y2="40.715" width="0.3" layer="1"/>
 </signal>
-<signal name="OLED_RST" class="2">
+<signal name="LCD_RST" class="2">
 <contactref element="LCD" pad="29_!RET!"/>
 <contactref element="R1" pad="2"/>
@@
 <wire x1="20.05" y1="28.95" x2="18.52" y2="30.48" width="0.3" layer="1"/>
 </signal>
-<signal name="OLED_!D!/C" class="2">
+<signal name="LCD_!D!/C" class="2">
 <contactref element="LCD" pad="28_A0(RS)"/>
 <via x="32.5" y="56" extent="1-16" drill="0.35"/>
@@
 <wire x1="34" y1="42.75" x2="34" y2="46.5" width="0.3" layer="1"/>
 </signal>
-<signal name="LED_BACKLIGHT_GREEN_GATE" class="2">
+<signal name="LCD_BACKLIGHT_GREEN_GATE" class="2">
 <contactref element="IC5" pad="27_PB15"/>
 <contactref element="IC3" pad="1_G1"/>
@@
 <wire x1="29.8" y1="31" x2="35.2" y2="31" width="0.3" layer="1"/>
 </signal>
-<signal name="LED_BACKLIGHT_IR_GATE" class="2">
+<signal name="LCD_BACKLIGHT_IR_GATE" class="2">
 <contactref element="IC5" pad="26_PB14"/>
 <contactref element="IC3" pad="3_G2"/>
@@
 <wire x1="46" y1="41.95" x2="46" y2="42.25" width="0.3" layer="1"/>
 </signal>
-<signal name="BACKLIGHT_GREEN_DRAIN" class="2">
+<signal name="LCD_BACKLIGHT_GREEN_DRAIN" class="2">
 <contactref element="IC3" pad="6_D1"/>
 <via x="35.25" y="28.75" extent="1-16" drill="0.35"/>
@@
 <wire x1="50.45" y1="40.75" x2="50.5" y2="40.8" width="0.3" layer="16"/>
 </signal>
-<signal name="BACKLIGHT_IR_DRAIN" class="2">
+<signal name="LCD_BACKLIGHT_IR_DRAIN" class="2">
 <contactref element="IC3" pad="4_D2"/>
 <via x="33.75" y="28.75" extent="1-16" drill="0.35"/>
