File: FLC-148 - LED & Keypad panel/FLC-148 LED & Keypad panel.brd (EAGLE design)
At the start: 52 x 73.8 mm, 74 parts, among them IC1 MAX6818, IC2 MAX6818, IC3 NTGD3148NT1G, IC4 NTGD3148NT1G, IC5 STM32G071CBU6, IC6 ECS-480-10-33B-CKM-TR, J1 FTSH-107-01-L-DV-K-A

Commit message: - renamed pins to be in sync with HW test script
Connections:
- net ALT_IN renamed KEYPAD_ALT_IN
- net ALT_OUT renamed KEYPAD_ALT_OUT_PIN
- net DOWN_IN renamed KEYPAD_DOWN_IN
- net DOWN_OUT renamed KEYPAD_DOWN_OUT_PIN
- net ENT_IN renamed KEYPAD_ENT_IN
- net ENT_OUT renamed KEYPAD_ENT_OUT_PIN
- net ESC_IN renamed KEYPAD_ESC_IN
- net ESC_OUT renamed KEYPAD_ESC_OUT_PIN
- net FN1_IN renamed SIDEPANEL_FN1_IN
- net FN1_OUT renamed SIDEPANEL_FN1_OUT_PIN
- net FN2_IN renamed SIDEPANEL_FN2_IN
- net FN2_OUT renamed SIDEPANEL_FN2_OUT_PIN
- net GR_IN renamed KEYPAD_GR_IN
- net GR_OUT renamed KEYPAD_GR_OUT_PIN
- net MODE_IN renamed KEYPAD_MODE_IN
- net MODE_OUT renamed KEYPAD_MODE_OUT_PIN
- net OLED_!D!/C renamed LCD_DC_PIN
- net OLED_BACKLIGHT_GREEN_GATE renamed LCD_BACKLIGHT_GREEN_GATE_PIN
- net OLED_BACKLIGHT_IR_GATE renamed LCD_BACKLIGHT_IR_GATE_PIN
- net OLED_RST renamed LCD_RST_PIN
- net OSC_IN renamed MCU_OSC_IN_PIN
- net OSC_OUT renamed MCU_OSC_OUT_PIN
- net PIN_CP1 renamed KEYPAD_CP1_PIN
- net PIN_CP2 renamed KEYPAD_CP2_PIN
- net PIN_CP3 renamed KEYPAD_CP3_PIN
- net PIN_CP4 renamed KEYPAD_CP4_PIN
- net PIN_CP5 renamed KEYPAD_CP5_PIN
- net PTT_IN renamed SIDEPANEL_PTT_IN
- net PTT_OUT renamed SIDEPANEL_PTT_OUT_PIN
- net SPI_OLED_MOSI renamed SPI_LCD_MOSI_PIN
- net SPI_OLED_SCK renamed SPI_LCD_SCK_PIN
- net SPI_OLED_SS renamed SPI_LCD_SS_PIN
- net SQL_IN renamed SIDEPANEL_SQL_IN
- net SQL_OUT renamed SIDEPANEL_SQL_OUT_PIN
- net SWDCLK renamed MCU_SWD_CLK_PIN
- net SWDIO renamed MCU_SWD_IO_PIN
- net UP_IN renamed KEYPAD_UP_IN
- net UP_OUT renamed KEYPAD_UP_OUT_PIN
- net WAKEUP renamed MCU_WAKEUP_PIN

Commit message: - added 10k pulldown to gate pins of illumination FETs, still needs routing
Connections:
- net GND: now also R3.P$4, R3.P$5, R3.P$6
- net KEYPAD_BACKLIGHT_IR_GATE: now also R3.P$11
- net LCD_BACKLIGHT_GREEN_GATE_PIN: now also R3.P$12
- net LCD_BACKLIGHT_IR_GATE_PIN: now also R3.P$13

Commit message: - renamed MCU_KEYPAD_INTERRUPT to MCU_TO_KEYPAD_INT - in schematic added button names for LED associated with a button
Connections:
- net MCU_KEYPAD_INTERRUPT renamed MCU_TO_KEYPAD_INT
Changed lines of the file:
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@@
 <grid distance="0.25" unitdist="mm" unit="mm" style="dots" multiple="1" display="yes" altdistance="0.05" altunitdist="mm" altunit="mm"/>
 <layers>
-<layer number="1" name="Top" color="4" fill="1" visible="yes" active="yes"/>
+<layer number="1" name="Top" color="4" fill="1" visible="no" active="yes"/>
 <layer number="2" name="Route2" color="16" fill="1" visible="no" active="yes"/>
 <layer number="3" name="Route3" color="17" fill="1" visible="no" active="no"/>
@@
 <layer number="14" name="Route14" color="22" fill="1" visible="no" active="no"/>
 <layer number="15" name="Route15" color="23" fill="1" visible="no" active="yes"/>
-<layer number="16" name="Bottom" color="1" fill="1" visible="no" active="yes"/>
+<layer number="16" name="Bottom" color="1" fill="1" visible="yes" active="yes"/>
 <layer number="17" name="Pads" color="2" fill="1" visible="yes" active="yes"/>
 <layer number="18" name="Vias" color="2" fill="1" visible="yes" active="yes"/>
 <layer number="19" name="Unrouted" color="6" fill="1" visible="yes" active="yes"/>
 <layer number="20" name="Dimension" color="24" fill="1" visible="yes" active="yes"/>
-<layer number="21" name="tPlace" color="7" fill="1" visible="yes" active="yes"/>
-<layer number="22" name="bPlace" color="7" fill="1" visible="no" active="yes"/>
-<layer number="23" name="tOrigins" color="15" fill="1" visible="yes" active="yes"/>
-<layer number="24" name="bOrigins" color="15" fill="1" visible="no" active="yes"/>
-<layer number="25" name="tNames" color="7" fill="1" visible="yes" active="yes"/>
-<layer number="26" name="bNames" color="7" fill="1" visible="no" active="yes"/>
+<layer number="21" name="tPlace" color="7" fill="1" visible="no" active="yes"/>
+<layer number="22" name="bPlace" color="7" fill="1" visible="yes" active="yes"/>
+<layer number="23" name="tOrigins" color="15" fill="1" visible="no" active="yes"/>
+<layer number="24" name="bOrigins" color="15" fill="1" visible="yes" active="yes"/>
+<layer number="25" name="tNames" color="7" fill="1" visible="no" active="yes"/>
+<layer number="26" name="bNames" color="7" fill="1" visible="yes" active="yes"/>
 <layer number="27" name="tValues" color="7" fill="1" visible="no" active="yes"/>
 <layer number="28" name="bValues" color="7" fill="1" visible="no" active="yes"/>
-<layer number="29" name="tStop" color="7" fill="3" visible="yes" active="yes"/>
-<layer number="30" name="bStop" color="7" fill="6" visible="no" active="yes"/>
+<layer number="29" name="tStop" color="7" fill="3" visible="no" active="yes"/>
+<layer number="30" name="bStop" color="7" fill="6" visible="yes" active="yes"/>
 <layer number="31" name="tCream" color="7" fill="4" visible="no" active="yes"/>
 <layer number="32" name="bCream" color="7" fill="5" visible="no" active="yes"/>
@@
 <layer number="37" name="tTest" color="7" fill="1" visible="no" active="yes"/>
 <layer number="38" name="bTest" color="7" fill="1" visible="no" active="yes"/>
-<layer number="39" name="tKeepout" color="4" fill="11" visible="yes" active="yes"/>
-<layer number="40" name="bKeepout" color="1" fill="11" visible="no" active="yes"/>
-<layer number="41" name="tRestrict" color="4" fill="10" visible="yes" active="yes"/>
-<layer number="42" name="bRestrict" color="1" fill="10" visible="no" active="yes"/>
+<layer number="39" name="tKeepout" color="4" fill="11" visible="no" active="yes"/>
+<layer number="40" name="bKeepout" color="1" fill="11" visible="yes" active="yes"/>
+<layer number="41" name="tRestrict" color="4" fill="10" visible="no" active="yes"/>
+<layer number="42" name="bRestrict" color="1" fill="10" visible="yes" active="yes"/>
 <layer number="43" name="vRestrict" color="2" fill="10" visible="yes" active="yes"/>
 <layer number="44" name="Drills" color="7" fill="1" visible="no" active="yes"/>
@@
 <layer number="49" name="Reference" color="7" fill="1" visible="no" active="yes"/>
 <layer number="50" name="dxf" color="7" fill="1" visible="no" active="no"/>
-<layer number="51" name="tDocu" color="7" fill="1" visible="yes" active="yes"/>
-<layer number="52" name="bDocu" color="7" fill="1" visible="no" active="yes"/>
+<layer number="51" name="tDocu" color="7" fill="1" visible="no" active="yes"/>
+<layer number="52" name="bDocu" color="7" fill="1" visible="yes" active="yes"/>
 <layer number="53" name="tGND_GNDA" color="7" fill="1" visible="no" active="no"/>
 <layer number="54" name="bGND_GNDA" color="7" fill="1" visible="no" active="no"/>
@@
 <wire x1="31" y1="53" x2="32.25" y2="54.25" width="0.3" layer="16"/>
 </signal>
-<signal name="MCU_KEYPAD_INTERRUPT" class="2">
+<signal name="MCU_TO_KEYPAD_INT" class="2">
 <contactref element="MCU" pad="6_PD9"/>
 <wire x1="27.75" y1="18.96" x2="27.75" y2="19.5" width="0.3" layer="1"/>
