File: FLC-148 - LED & Keypad panel/FLC-148 LED & Keypad panel.sch (EAGLE design)
At the start: 76 parts, among them IC1 MAX6818, IC2 MAX6818, IC3 NTGD3148NT1G, IC4 NTGD3148NT1G, IC5 STM32G071CBU6, IC6 ECS-480-10-33B-CKM-TR, J1 FTSH-107-01-L-DV-K-A

Commit message: start of rev.2 board - the LCD D/C signal wasn't routed - pulldown resistors are likely needed for LED gate control - boot0 likely needs to be tied to GND
Connections:
- net BACKLIGHT_GREEN_DRAIN renamed LCD_BACKLIGHT_GREEN_DRAIN
- net BACKLIGHT_IR_DRAIN renamed LCD_BACKLIGHT_IR_DRAIN
- net LED_BACKLIGHT_GREEN_GATE renamed LCD_BACKLIGHT_GREEN_GATE
- net LED_BACKLIGHT_IR_GATE renamed LCD_BACKLIGHT_IR_GATE
- net OLED_!D!/C renamed LCD_!D!/C
- net OLED_RST renamed LCD_RST
Other:
- note added: "TODO: route D/C line"
Changed lines of the file:
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@@
 <text x="662.94" y="-91.44" size="1.778" layer="98">wakeup</text>
 <text x="662.94" y="7.62" size="1.778" layer="98">wakeup</text>
-<text x="685.8" y="-127" size="1.778" layer="98">TODO: tie boot0 to gnd</text>
+<text x="815.34" y="-33.02" size="3.81" layer="98" rot="R270">TODO: tie boot0 to gnd</text>
 <text x="132.08" y="-15.24" size="1.778" layer="90">BOOT0 pin</text>
+<text x="63.5" y="-5.08" size="3.81" layer="98" rot="R270">TODO: route D/C line</text>
 </plain>
 <instances>
@@
 </segment>
 </net>
-<net name="OLED_RST" class="2">
+<net name="LCD_RST" class="2">
 <segment>
 <pinref part="LCD" gate="G$1" pin="!RET!_29"/>
@@
 </segment>
 </net>
-<net name="OLED_!D!/C" class="2">
+<net name="LCD_!D!/C" class="2">
 <segment>
 <pinref part="LCD" gate="G$1" pin="A0(RS)_28"/>
@@
 </segment>
 </net>
-<net name="LED_BACKLIGHT_GREEN_GATE" class="2">
+<net name="LCD_BACKLIGHT_GREEN_GATE" class="2">
 <segment>
 <pinref part="IC5" gate="G$1" pin="SPI2_MOSI,TIM1_CH3N,TIM15_CH1N,TIM15_CH2,EVENTOUT,UCPD1_CC2,RTC_REFIN-PB15"/>
@@
 </segment>
 </net>
-<net name="LED_BACKLIGHT_IR_GATE" class="2">
+<net name="LCD_BACKLIGHT_IR_GATE" class="2">
 <segment>
 <pinref part="IC5" gate="G$1" pin="SPI2_MISO,UCPD1_FRSTX,TIM1_CH2N,USART3_RTS_DE_CK,TIM15_CH1,I2C2_SDA,EVENTOUT-PB14"/>
@@
 </segment>
 </net>
-<net name="BACKLIGHT_GREEN_DRAIN" class="2">
+<net name="LCD_BACKLIGHT_GREEN_DRAIN" class="2">
 <segment>
 <pinref part="IC3" gate="G$1" pin="6_D1"/>
@@
 </segment>
 </net>
-<net name="BACKLIGHT_IR_DRAIN" class="2">
+<net name="LCD_BACKLIGHT_IR_DRAIN" class="2">
 <segment>
 <pinref part="IC3" gate="G$1" pin="4_D2"/>
