File: FLC-148 - LED & Keypad panel/FLC-148 LED & Keypad panel.sch (EAGLE design)
At the start: 74 parts, among them IC1 MAX6818, IC2 MAX6818, IC3 NTGD3148NT1G, IC4 NTGD3148NT1G, IC5 STM32G071CBU6, IC6 ECS-480-10-33B-CKM-TR, J1 FTSH-107-01-L-DV-K-A

Commit message: - more todo updates - added ground vias
Other:
- note added: "TODO - logic gates: add logic OR gates to pushbutton switches & tie to wakeup pin so that microcontroller can be waken up on key press - quad FET: replace 2 dual FETs with one quad fet component - output debouncing: add debouncing circuitry to rotary encoder A and B output channels - pulldown: add 10k pulldown to FET gate pins - conector rework: pick different connectors & orient them better"
- note added: "TODO: connector rework"
- note removed: "TODO - logic gates: add logic OR gates to pushbutton switches & tie to wakeup pin so that microcontroller can be waken up on key press - quad FET: replace 2 dual FETs with one quad fet component - output debouncing: add debouncing circuitry to rotary encoder A and B output channels - pulldown: add 10k pulldown to FET gate pins -"
Changed lines of the file:
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@@
 - output debouncing: add debouncing circuitry to rotary encoder A and B output channels
 - pulldown: add 10k pulldown to FET gate pins
-- </text>
+- conector rework: pick different connectors &amp; orient them better</text>
 <text x="55.88" y="33.02" size="1.778" layer="94">TODO: output debouncing</text>
 <text x="396.24" y="-175.26" size="1.778" layer="94">TODO: pulldown</text>
@@
 <text x="396.24" y="-200.66" size="1.778" layer="94">TODO: pulldown</text>
 <text x="706.12" y="7.62" size="1.778" layer="98">WKUP6</text>
+<text x="5.08" y="48.26" size="1.778" layer="94">TODO: connector rework</text>
 </plain>
 <instances>
