File: FLC-148 - LED & Keypad panel/FLC-148 LED & Keypad panel.sch (EAGLE design)
At the start: 74 parts, among them IC1 MAX6818, IC2 MAX6818, IC3 NTGD3148NT1G, IC4 NTGD3148NT1G, IC5 STM32G071CBU6, IC6 ECS-480-10-33B-CKM-TR, J1 FTSH-107-01-L-DV-K-A

Commit message: - renamed pins to be in sync with HW test script
Connections:
- net ALT_IN renamed KEYPAD_ALT_IN
- net ALT_OUT renamed KEYPAD_ALT_OUT_PIN
- net DOWN_IN renamed KEYPAD_DOWN_IN
- net DOWN_OUT renamed KEYPAD_DOWN_OUT_PIN
- net ENT_IN renamed KEYPAD_ENT_IN
- net ENT_OUT renamed KEYPAD_ENT_OUT_PIN
- net ESC_IN renamed KEYPAD_ESC_IN
- net ESC_OUT renamed KEYPAD_ESC_OUT_PIN
- net FN1_IN renamed SIDEPANEL_FN1_IN
- net FN1_OUT renamed SIDEPANEL_FN1_OUT_PIN
- net FN2_IN renamed SIDEPANEL_FN2_IN
- net FN2_OUT renamed SIDEPANEL_FN2_OUT_PIN
- net GR_IN renamed KEYPAD_GR_IN
- net GR_OUT renamed KEYPAD_GR_OUT_PIN
- net MODE_IN renamed KEYPAD_MODE_IN
- net MODE_OUT renamed KEYPAD_MODE_OUT_PIN
- net OLED_!D!/C renamed LCD_DC_PIN
- net OLED_BACKLIGHT_GREEN_GATE renamed LCD_BACKLIGHT_GREEN_GATE_PIN
- net OLED_BACKLIGHT_IR_GATE renamed LCD_BACKLIGHT_IR_GATE_PIN
- net OLED_RST renamed LCD_RST_PIN
- net OSC_IN renamed MCU_OSC_IN_PIN
- net OSC_OUT renamed MCU_OSC_OUT_PIN
- net PIN_CP1 renamed KEYPAD_CP1_PIN
- net PIN_CP2 renamed KEYPAD_CP2_PIN
- net PIN_CP3 renamed KEYPAD_CP3_PIN
- net PIN_CP4 renamed KEYPAD_CP4_PIN
- net PIN_CP5 renamed KEYPAD_CP5_PIN
- net PTT_IN renamed SIDEPANEL_PTT_IN
- net PTT_OUT renamed SIDEPANEL_PTT_OUT_PIN
- net SPI_OLED_MOSI renamed SPI_LCD_MOSI_PIN
- net SPI_OLED_SCK renamed SPI_LCD_SCK_PIN
- net SPI_OLED_SS renamed SPI_LCD_SS_PIN
- net SQL_IN renamed SIDEPANEL_SQL_IN
- net SQL_OUT renamed SIDEPANEL_SQL_OUT_PIN
- net SWDCLK renamed MCU_SWD_CLK_PIN
- net SWDIO renamed MCU_SWD_IO_PIN
- net UP_IN renamed KEYPAD_UP_IN
- net UP_OUT renamed KEYPAD_UP_OUT_PIN
- net WAKEUP renamed MCU_WAKEUP_PIN
Other:
- note added: "TODO - MCU wakeup & logic gates: add logic OR gates to pushbutton switches & tie to wakeup pin so that microcontroller can be waken up on key press - quad FET: replace 2 dual FETs with one quad fet component - output debouncing: add debouncing circuitry to rotary encoder A and B output channels - pulldown: add 10k pulldown to FET gate pins - conector rework: pick different connectors & orient the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"
- note added: "TODO: MCU wakeup"
- note removed: "TODO - logic gates: add logic OR gates to pushbutton switches & tie to wakeup pin so that microcontroller can be waken up on key press - quad FET: replace 2 dual FETs with one quad fet component - output debouncing: add debouncing circuitry to rotary encoder A and B output channels - pulldown: add 10k pulldown to FET gate pins - conector rework: pick different connectors & orient them better"
- moved on the sheet: R4

Commit message: - added 10k pulldown to gate pins of illumination FETs, still needs routing
Connections:
- net GND: now also R3.P$4, R3.P$5, R3.P$6
- net KEYPAD_BACKLIGHT_IR_GATE: now also R3.P$11
- net LCD_BACKLIGHT_GREEN_GATE_PIN: now also R3.P$12
- net LCD_BACKLIGHT_IR_GATE_PIN: now also R3.P$13
Other:
- note added: "EXTI12"
- note added: "EXTI3"
- note added: "TIM2_CH3"
- note added: "TIM2_CH4"
- note added: "TODO - MCU wakeup & logic gates: add logic OR gates to pushbutton switches & tie to wakeup pin so that microcontroller can be waken up on key press - quad FET: replace 2 dual FETs with one quad fet component - output debouncing: add debouncing circuitry to rotary encoder A and B output channels - pulldown: route 10k pulldown to FET gate pins - conector rework: pick different connectors & orient t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"
- note added: "TODO: EXTI conflict"
- note removed: "TODO - MCU wakeup & logic gates: add logic OR gates to pushbutton switches & tie to wakeup pin so that microcontroller can be waken up on key press - quad FET: replace 2 dual FETs with one quad fet component - output debouncing: add debouncing circuitry to rotary encoder A and B output channels - pulldown: add 10k pulldown to FET gate pins - conector rework: pick different connectors & orient the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"
Changed lines of the file:
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@@
 - quad FET: replace 2 dual FETs with one quad fet component
 - output debouncing: add debouncing circuitry to rotary encoder A and B output channels
-- pulldown: add 10k pulldown to FET gate pins
-- conector rework: pick different connectors &amp; orient them better</text>
+- pulldown: route 10k pulldown to FET gate pins
+- conector rework: pick different connectors &amp; orient them better
+- EXTI conflict: PB6 and PC6 both have EXTI6</text>
 <text x="55.88" y="33.02" size="1.778" layer="94">TODO: output debouncing</text>
 <text x="396.24" y="-175.26" size="1.778" layer="94">TODO: pulldown</text>
@@
 <text x="5.08" y="48.26" size="1.778" layer="94">TODO: connector rework</text>
 <text x="134.62" y="40.64" size="1.778" layer="94">TODO: MCU wakeup</text>
+<text x="723.9" y="-38.1" size="1.9304" layer="94">TODO: EXTI conflict</text>
+<text x="708.66" y="10.16" size="1.9304" layer="94">TODO: EXTI conflict</text>
+<text x="683.26" y="-63.5" size="1.778" layer="98">EXTI12</text>
+<text x="683.26" y="-88.9" size="1.778" layer="98">EXTI3</text>
+<text x="683.26" y="-68.58" size="1.778" layer="98">TIM2_CH3</text>
+<text x="683.26" y="-66.04" size="1.778" layer="98">TIM2_CH4</text>
+<text x="193.04" y="43.18" size="1.778" layer="94">TODO: pulldown</text>
 </plain>
 <instances>
@@
 <wire x1="167.64" y1="-48.26" x2="167.64" y2="-50.8" width="0.1524" layer="91"/>
 <label x="167.64" y="-50.8" size="1.778" layer="95"/>
+</segment>
+<segment>
+<pinref part="R3" gate="G$1" pin="P$4"/>
+<wire x1="193.04" y1="60.96" x2="187.96" y2="60.96" width="0.1524" layer="91"/>
+<label x="187.96" y="60.96" size="1.778" layer="95" rot="R180"/>
+</segment>
+<segment>
+<pinref part="R3" gate="G$1" pin="P$5"/>
+<wire x1="193.04" y1="58.42" x2="187.96" y2="58.42" width="0.1524" layer="91"/>
+<label x="187.96" y="58.42" size="1.778" layer="95" rot="R180"/>
+</segment>
+<segment>
+<pinref part="R3" gate="G$1" pin="P$6"/>
+<wire x1="193.04" y1="55.88" x2="187.96" y2="55.88" width="0.1524" layer="91"/>
+<label x="187.96" y="55.88" size="1.778" layer="95" rot="R180"/>
 </segment>
 </net>
@@
 <label x="358.14" y="-180.34" size="1.778" layer="95"/>
 </segment>
+<segment>
+<pinref part="R3" gate="G$1" pin="P$12"/>
+<wire x1="208.28" y1="58.42" x2="213.36" y2="58.42" width="0.1524" layer="91"/>
+<label x="213.36" y="58.42" size="1.778" layer="95"/>
+</segment>
 </net>
 <net name="LCD_BACKLIGHT_IR_GATE_PIN" class="2">
@@
 <wire x1="350.52" y1="-175.26" x2="358.14" y2="-175.26" width="0.1524" layer="91"/>
 <label x="358.14" y="-175.26" size="1.778" layer="95"/>
+</segment>
+<segment>
+<pinref part="R3" gate="G$1" pin="P$13"/>
+<wire x1="208.28" y1="60.96" x2="213.36" y2="60.96" width="0.1524" layer="91"/>
+<label x="213.36" y="60.96" size="1.778" layer="95"/>
 </segment>
 </net>
@@
 <label x="358.14" y="-200.66" size="1.778" layer="95"/>
 </segment>
-</net>
+<segment>
+<pinref part="R3" gate="G$1" pin="P$11"/>
+<wire x1="208.28" y1="55.88" x2="213.36" y2="55.88" width="0.1524" layer="91"/>
+<label x="213.36" y="55.88" size="1.778" layer="95"/>
+</segment>
+</net>
